Commit message: ROS2 graph: /World root, elbow-only position control; fix camera_mount URDF joints

File: assets/urdf/urdf/volcaniarm.urdf (robot description, URDF)
Before this commit: robot volcaniarm, 23 links, 22 joints
Joints:
- joint camera_mount_linear_joint: type prismatic -> fixed
- joint camera_mount_rev_joint: type revolute -> fixed

Commit message: Sync camera chain to ROS URDF + align sensor prim to optical frame
URDF (assets/urdf/urdf/volcaniarm.urdf):
- camera_mount_linear_joint xyz X: 0.405 -> 0.25
- camera_mount_rev_joint pitch: 0.212 -> 1.3
- camera_joint xyz: (-2.4e-5, 0, 0.016) -> (0.016, 0, 0)
- camera_joint rpy: (0, -0.0135, 0) -> (pi, 0, 0)
- camera_mount_rev_link visual origin rpy: (0,0,0) -> (0, pi/2, 0)
- camera_link visual origin rpy: (0,0,0) -> (0, pi/2, 0)
- Add camera_link_optical link + camera_optical_joint
- Drop axis/limit/dynamics from fixed camera joints (ignored on fixed
  joints, not present in the ROS URDF)
All values match the ROS xacro defaults so the two sims agree on the
camera mount position, pitch angle, and optical frame chain.

add_ros2_graph.py:
- Apply rpy=(90, 0, -90) to the USD camera sensor prim. This aligns
  the sensor axes with camera_color_optical_frame (ROS convention:
  +X right, +Y down, +Z forward) AND flips USD's default -Z look
  direction into the +Z the optical frame expects, so image/pointcloud
  published on /camera/color/... carry a frame_id that resolves
  consistently in RViz.

File: assets/urdf/urdf/volcaniarm.urdf (robot description, URDF)
Before this commit: robot volcaniarm, 23 links, 22 joints
Links:
- added link camera_link_optical
Joints:
- added joint camera_optical_joint: type fixed, parent camera_link, child camera_link_optical, origin xyz=0 0 0 rpy=-1.5708 0 -1.5708
- joint camera_joint: axis 0 0 0 -> (none); origin xyz=-2.37779715432929E-05 0 0.0160004150359285 rpy=0 -0.0135473024600912 0 -> xyz=0.0160004150359285 0 0 rpy=3.14159 0 0
- joint camera_mount_linear_joint: axis 1 0 0 -> (none); limit lower=-0.3 upper=0.3 effort=10 velocity=10 -> (none); origin xyz=0.405353761834025 0 0.039999999999992 rpy=0 0 0 -> xyz=0.25 0 0.039999999999992 rpy=0 0 0
- joint camera_mount_rev_joint: axis 0 1 0 -> (none); limit lower=-3.14 upper=3.14 effort=10 velocity=10 -> (none); origin xyz=0.192000000000008 0 -0.0290000000000052 rpy=3.14159265358979 0.211904134210419 3.14159265358979 -> xyz=0.192000000000008 0 -0.0290000000000052 rpy=3.14159265358979 1.3 3.14159265358979

Commit message: Elbow joint limits from CAD: right [45,160]deg, left [-160,-45]deg; center init + narrow reset

File: assets/urdf/urdf/volcaniarm.urdf (robot description, URDF)
Before this commit: robot volcaniarm, 24 links, 23 joints
Joints:
- joint volcaniarm_left_elbow_joint: limit lower=-3.14 upper=3.14 effort=10 velocity=10 -> lower=-2.792526803190927 upper=-0.7853981633974483 effort=10 velocity=10
- joint volcaniarm_right_elbow_joint: limit lower=-3.14 upper=3.14 effort=10 velocity=10 -> lower=0.7853981633974483 upper=2.792526803190927 effort=10 velocity=10

Commit message: Baseline reset: revert joint limits/init/reset/target-Z, reach-only rewards

File: assets/urdf/urdf/volcaniarm.urdf (robot description, URDF)
Before this commit: robot volcaniarm, 24 links, 23 joints
Joints:
- joint volcaniarm_left_elbow_joint: limit lower=-2.792526803190927 upper=-0.7853981633974483 effort=10 velocity=10 -> lower=-3.14 upper=3.14 effort=10 velocity=10
- joint volcaniarm_right_elbow_joint: limit lower=0.7853981633974483 upper=2.792526803190927 effort=10 velocity=10 -> lower=-3.14 upper=3.14 effort=10 velocity=10
