Commit message: scripts: generate Isaac URDF from ws xacro (sync_urdf.py); regen assets/urdf
Kills the hand-maintained fork. Notable in the regen: 6 mesh STLs had
silently drifted from the ws; ee closure z adopts the ws 0.6225 (fork had
0.62243); palette colors now flow from the ws materials.xacro.

File: assets/urdf/urdf/volcaniarm.urdf (robot description, URDF)
Before this commit: robot volcaniarm, 24 links, 23 joints
Links:
- link camera_mount_linear_link: mass 0 -> 0.1
Joints:
- added joint world_to_base: type fixed, parent world, child base_link, origin xyz=0 0 0.98 rpy=0 0 3.14159
- joint camera_joint: origin xyz=0.0160004150359285 0 0 rpy=3.14159 0 0 -> xyz=0.0160004150359285 0.0 0.0 rpy=3.14159 0.0 0.0
- joint fl_caster_wheel_joint: axis 0 0 0 -> (none)
- joint fl_caster_wheel_mount_joint: axis 0 0 0 -> (none)
- joint fl_table_leg_joint: axis 0 0 0 -> (none)
- joint fr_caster_wheel_joint: axis 0 0 0 -> (none)
- joint fr_caster_wheel_mount_joint: axis 0 0 0 -> (none)
- joint fr_table_leg_joint: axis 0 0 0 -> (none)
- joint left_ee_joint: axis 0 0 0 -> (none); origin xyz=0 0 0.62243 rpy=0 0 0 -> xyz=0 0 0.6225 rpy=0 0 0
- joint right_ee_joint: axis 0 0 0 -> (none); origin xyz=0 0 0.62243 rpy=0 0 0 -> xyz=0 0 0.6225 rpy=0 0 0
- joint rl_caster_wheel_joint: axis 0 0 0 -> (none)
- joint rl_caster_wheel_mount_joint: axis 0 0 0 -> (none)
- joint rl_table_leg_joint: axis 0 0 0 -> (none)
- joint rr_caster_wheel_joint: axis 0 0 0 -> (none)
- joint rr_caster_wheel_mount_joint: axis 0 0 0 -> (none)
- joint rr_table_leg_joint: axis 0 0 0 -> (none)
- joint volcaniarm_base_joint: axis 0 0 0 -> (none)
- joint volcaniarm_left_arm_joint: axis -1 0 0 -> 1 0 0; origin xyz=0.00399999999997247 0.0200000000000011 0.416213203435623 rpy=-1.70529629561765 0 0 -> xyz=0.004 0.02 0.41621 rpy=-1.7053 0 0
- joint volcaniarm_left_elbow_joint: origin xyz=0.285000000000036 -0.214999999999991 0.0632000000000055 rpy=0.785398163397457 0 0 -> xyz=0.285 -0.215 0.0632 rpy=0.7854 0 0
- joint volcaniarm_right_elbow_joint: origin xyz=0.289000000000013 0.215 0.0632000000000104 rpy=-0.785398163397448 0 0 -> xyz=0.289 0.215 0.0632 rpy=-0.7854 0 0

Commit message: sync_urdf: remove joints on both sides of stripped links (dangling world_to_base crashed the URDF parser); verify joint refs

File: assets/urdf/urdf/volcaniarm.urdf (robot description, URDF)
Before this commit: robot volcaniarm, 24 links, 24 joints
Joints:
- removed joint world_to_base
